File: hardware/we_ssr_control/we_ssr_control.kicad_pcb (KiCad board)
At the start: 2 copper layers, 65 x 90 mm, 50 parts, among them Q1 IRF4905PBF, U1 WeMos_D1_mini

Commit message: Merged all symbol, 3dmodel, and footprint changes
Parts:
- RZ1: footprint Resistor_SMD:R_0805_2012Metric -> Resistor_SMD:R_0603_1608Metric
- moved RZ1 0.09 mm to (100.8, 79.2)
Connections:
- net +VDC renamed /Power Management/VDC
- U1 pad 1: (no net) -> unconnected-(U1-Pad1)
- U1 pad 15: (no net) -> unconnected-(U1-Pad15)
- U1 pad 16: (no net) -> unconnected-(U1-Pad16)
- U1 pad 2: (no net) -> unconnected-(U1-Pad2)
- U1 pad 8: (no net) -> unconnected-(U1-Pad8)
Routing:
- net GNDPWR: vias 84 -> 91
