File: hardware/we_ssr_control/we_ssr_control.kicad_pcb (KiCad board)
At the start: 2 copper layers, 65 x 90 mm, 50 parts, among them Q1 IRF4905PBF, U1 WeMos_D1_mini

Commit message: Power supply changes plus misc.
Parts:
- removed #LOGO3: 6, Symbol:KiCad-Logo_8mm_SilkScreen
- removed REG1: LM7805, Package_TO_SOT_SMD:SOT-223
- removed RZ1: 100k, Resistor_SMD:R_0603_1608Metric
- added C10: 4u7, Capacitor_SMD:C_0805_2012Metric, F.Cu at (91.0, 66.2)
- added C11: 100n, Capacitor_SMD:C_0603_1608Metric, F.Cu at (87.0, 75.8)
- added C3: 220n, Capacitor_SMD:C_0603_1608Metric, F.Cu at (95.7, 70.4)
- added C4: 1u, Capacitor_SMD:C_0603_1608Metric, F.Cu at (97.7, 59.9)
- added C5: 100n, Capacitor_SMD:C_0603_1608Metric, F.Cu at (92.5, 61.0)
- added C6: 4u7, Capacitor_SMD:C_0805_2012Metric, F.Cu at (91.0, 76.5)
- added C7: 4u7, Capacitor_SMD:C_0805_2012Metric, F.Cu at (91.0, 73.8)
- added C8: 4u7, Capacitor_SMD:C_0805_2012Metric, F.Cu at (91.0, 71.2)
- added C9: 4u7, Capacitor_SMD:C_0805_2012Metric, F.Cu at (91.0, 68.7)
- added L1: 2u2, Inductor_SMD:L_1008_2520Metric, F.Cu at (90.0, 63.0)
- added R1: 100k, Resistor_SMD:R_0603_1608Metric, F.Cu at (106.6, 66.2)
- added R2: 100k, Resistor_SMD:R_0603_1608Metric, F.Cu at (97.0, 57.5)
- added R3: 100k, Resistor_SMD:R_0603_1608Metric, F.Cu at (100.0, 63.0)
- added R4: 24k9, Resistor_SMD:R_0603_1608Metric, F.Cu at (101.7, 63.0)
- added REF_KiCAD: KiCad-Logo2_5mm_SilkScreen, Symbol:KiCad-Logo2_5mm_SilkScreen, B.Cu at (92.9, 131.0)
- added U2: LMR33610BDDAR, Package_SO:Texas_HSOP-8-1EP_3.9x4.9mm_P1.27mm_ThermalVias, F.Cu at (96.3, 64.8)
- C1: value 330n -> 4u7
- C2: value 100n -> 4u7
- JL1, JS2: footprint Connector_PinHeader_1.00mm:PinHeader_1x02_P1.00mm_Vertical -> dragon_mobile:PinHeader_1x02_P1.00mm_Vertical
- Q1: value IRF4905PBF -> SQ3419EV-T1_GE3; footprint dragon_mobile:TO254P469X1042X1967-3P -> dragon_mobile:SOT95P284X110-6N
- QD1, QD2, QD3, QD4, QD5, QD6, QD7, QD8: footprint Package_TO_SOT_SMD:SOT-23 -> Package_TO_SOT_SMD:SOT-23-3
- RL1, RS1, RS2, RS3, RS4, RS5, RS6, RS7, RS8: value 270 -> 270R
- ZD1: value +10v Zener Diode -> 10V; footprint dragon_mobile:BZD27C10P-M3-08 -> Diode_SMD:D_0805_2012Metric
- moved ZD1 10.5 mm to (104.1, 67.1)
- moved C2 8.66 mm to (97.7, 70.5), turned to -90 degrees
- moved JS2 6.05 mm to (104.5, 76.8), turned to 90 degrees
- moved JP1 4.76 mm to (105.3, 60.3)
- moved C1 3.93 mm to (100.4, 70.5)
- moved Q1 3.70 mm to (104.7, 70.5), turned to 180 degrees
- moved RL1 1.52 mm to (105.2, 58.1), turned to 180 degrees
- moved LP1 0.92 mm to (105.2, 53.6)
- moved JL1 0.79 mm to (105.3, 56.0)
Connections:
- C2 pad 1: +5V -> /Power Management/VDC
- Q1 pad 1: Net-(Q1-Pad1) -> +BATT
- Q1 pad 3: /Power Management/VDC -> Net-(Q1-Pad3)
- U1 pad 1: unconnected-(U1-Pad1) -> /Power Management/PG
- ZD1 pad 2: Net-(Q1-Pad1) -> Net-(Q1-Pad3)
Routing:
- net /Power Management/PG: track 0.00 -> 52.2 mm, vias 0 -> 2
- net +5V: track 28.6 -> 49.1 mm, vias 0 -> 2
- net Net-(Q1-Pad1): track 6.61 -> 0.00 mm
- net +BATT: track 12.3 -> 7.23 mm, vias 0 -> 6
- net /Power Management/BOOT: track 0.00 -> 4.71 mm
- net Net-(Q1-Pad3): track 0.00 -> 3.89 mm
- net /Power Management/VCC: track 0.00 -> 3.82 mm
- net /Power Management/VDC: track 17.4 -> 13.6 mm
- net /Power Management/FB: track 0.00 -> 3.45 mm
- net GNDPWR: vias 91 -> 170
- added copper zone on B.Cu, net +BATT
- added copper zone on F.Cu, net +BATT
- added copper zone on F.Cu, net /Power Management/SW
Other:
- board text added: "v0.0.11"
- board text added: "© 2023 Michael Cummings"
- board text removed: "v0.0.10"
- board text removed: "© 2022 Michael Cummings"

Commit message: Pre KiCad 7.0.0 WIP
Parts:
- QD1, QD2, QD3, QD4, QD5, QD6, QD7, QD8: footprint Package_TO_SOT_SMD:SOT-23-3 -> dragon_mobile:2V7002KT1G
- moved #LOGO1 53.4 mm to (38.2, 71.7)
- moved #LOGO2 53.4 mm to (27.7, 65.7)
- moved QRCode1 53.4 mm to (31.2, 68.5)
- moved FID3 46.1 mm to (80.0, 100.0)
- moved H2 46.1 mm to (25.0, 100.0)
- moved REF_KiCAD 45.0 mm to (64.2, 96.3)
- moved S1 45.0 mm to (64.2, 97.7)
- moved C10 42.4 mm to (61.0, 36.1)
- moved C8 42.4 mm to (61.0, 41.2)
- moved QD5 42.4 mm to (55.6, 85.0)
- moved QD6 42.4 mm to (55.6, 81.0)
- moved QD7 42.4 mm to (55.6, 77.0)
- moved QD8 42.4 mm to (55.6, 73.0)
- moved C1 42.4 mm to (70.4, 40.5)
- moved C11 42.4 mm to (57.0, 45.8)
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Routing:
- net /Control Out/BANK_A.CNTL1: track 54.4 -> 0.00 mm, vias 2 -> 0
- net /Control Out/BANK_A.CNTL2: track 50.4 -> 0.00 mm, vias 2 -> 0
- net /WeMOS Control/IO5: track 52.8 -> 2.41 mm
- net /WeMOS Control/IO6: track 51.4 -> 2.41 mm
- net /WeMOS Control/IO7: track 49.9 -> 2.41 mm
- net /Control Out/BANK_A.CNTL3: track 46.4 -> 0.00 mm, vias 2 -> 0
- net /WeMOS Control/IO8: track 48.5 -> 2.41 mm
- net /Control Out/BANK_A.CNTL4: track 42.4 -> 0.00 mm, vias 2 -> 0
- net /WeMOS Control/IO4: track 44.4 -> 2.48 mm
- net /Control Out/BANK_B.CNTL8: track 40.3 -> 0.00 mm, vias 2 -> 0
- net /Control Out/BANK_B.CNTL7: track 36.3 -> 0.00 mm, vias 2 -> 0
- net /WeMOS Control/IO3: track 35.8 -> 2.48 mm
- net /Control Out/BANK_B.CNTL6: track 32.3 -> 0.00 mm, vias 2 -> 0
- net /Control Out/PwrIn2: track 30.1 -> 0.00 mm
- net /Control Out/BANK_B.CNTL5: track 28.2 -> 0.00 mm, vias 2 -> 0
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Other:
- board size 65 x 90 mm -> 65 x 85 mm
- board text added: "+BATT OUT1 OUT2 OUT3 OUT4"
- board text added: "0"
- board text added: "0 mm"
- board text added: "0.01 mm"
- board text added: "0.02"
- board text added: "0.035 mm"
- board text added: "1"
- board text added: "1 mm"
- board text added: "1.0900 mm"
- board text added: "3.3"
- board text added: "4.5"
- board text added: "B.Cu"
- board text added: "B.Mask"
- board text added: "B.Paste"
- board text added: "B.Silkscreen"
- board text added: "Bottom Silk Screen"
- board text added: "Bottom Solder Mask"
- board text added: "Bottom Solder Paste"
- board text added: "Color"
- board text added: "Dielectric 1"
- board text added: "Epsilon R"
- board text added: "F.Cu"
- board text added: "F.Mask"
- board text added: "F.Paste"
- board text added: "F.Silkscreen"
- board text added: "FR4"
- board text added: "Green"
- board text added: "Layer Name"
- board text added: "Loss Tangent"
- board text added: "Material"
- board text added: "Not specified"
- board text added: "OUT8 OUT7 OUT6 OUT5 +BATT"
- board text added: "Thickness (mm)"
- board text added: "Top Silk Screen"
- board text added: "Top Solder Mask"
- board text added: "Top Solder Paste"
- board text added: "Type"
- board text added: "White"
- board text added: "copper"
- board text added: "core"
- board text removed: "+BATT CNTL1 CNTL2 CNTL3 CNTL4"
- board text removed: "1.1600 mm"
- board text removed: "A1"
- board text removed: "A2"
- board text removed: "A3"
- board text removed: "A4"
- board text removed: "B5"
- board text removed: "B6"
- board text removed: "B7"
- board text removed: "B8"
- board text removed: "CNTL8 CNTL7 CNTL6 CNTL5 +BATT"
- board text removed: "H2"
- board text removed: "H3"
