File: hardware/we_ssr_control/wemos_control.kicad_sch (KiCad schematic)
At the start: 17 parts, among them U1 WeMos_D1_mini

Commit message: Merged all symbol, 3dmodel, and footprint changes
Connections:
- no-connect marks 1 -> 6
Changed lines of the file:
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@@
   (junction (at 78.74 137.16) (diameter 0) (color 0 0 0 0)
   )
+  (no_connect (at 17.78 68.58))
   (no_connect (at 38.1 66.04))
+  (no_connect (at 17.78 71.12))
+  (no_connect (at 17.78 66.04))
+  (no_connect (at 17.78 76.2))
+  (no_connect (at 17.78 73.66))
   (bus_entry (at 93.98 96.52) (size 2.54 -2.54)
     (stroke (width 0) (type default) (color 0 0 0 0))
@@
       (effects (font (size 1.27 1.27)) (justify left) hide)
     )
-    (property "Footprint" "dragon_mobile:WEMOS_D1_mini_light" (id 2) (at 27.94 105.41 0)
-      (effects (font (size 1.27 1.27)) hide)
-    )
-    (property "Datasheet" "https://wiki.wemos.cc/products:d1:d1_mini#documentation" (id 3) (at -19.05 105.41 0)
+    (property "Footprint" "dragon_mobile:WEMOS_D1_mini_light" (id 2) (at 27.94 113.03 0)
+      (effects (font (size 1.27 1.27)) hide)
+    )
+    (property "Datasheet" "https://wiki.wemos.cc/products:d1:d1_mini#documentation" (id 3) (at 27.94 117.094 0)
       (effects (font (size 1.27 1.27)) hide)
     )
@@
       (effects (font (size 1.27 1.27)) hide)
     )
+    (pin "1")
     (pin "10")
     (pin "11")
@@
     (pin "13")
     (pin "14")
+    (pin "15")
+    (pin "16")
+    (pin "2")
     (pin "3")
     (pin "4")
@@
     (pin "6")
     (pin "7")
+    (pin "8")
     (pin "9")
   )
