File: hardware/we_ssr_control/wemos_control.kicad_sch (KiCad schematic)
At the start: 18 parts, among them U1 WeMos_D1_mini

Commit message: Commit before removing git submodules
Changed lines of the file:
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@@
   (junction (at 89.154 48.26) (diameter 0) (color 0 0 0 0)
   )
+  (junction (at 88.9 93.98) (diameter 0) (color 0 0 0 0)
+  )
+  (junction (at 104.14 114.3) (diameter 0) (color 0 0 0 0)
+  )
+  (junction (at 101.6 68.58) (diameter 0) (color 0 0 0 0)
+  )
+  (junction (at 101.6 144.78) (diameter 0) (color 0 0 0 0)
+  )
+  (junction (at 101.6 99.06) (diameter 0) (color 0 0 0 0)
+  )
+  (junction (at 101.6 114.3) (diameter 0) (color 0 0 0 0)
+  )
+  (junction (at 101.6 160.02) (diameter 0) (color 0 0 0 0)
+  )
+  (junction (at 104.14 83.82) (diameter 0) (color 0 0 0 0)
+  )
+  (junction (at 104.14 160.02) (diameter 0) (color 0 0 0 0)
+  )
+  (junction (at 104.14 144.78) (diameter 0) (color 0 0 0 0)
+  )
+  (junction (at 88.9 109.22) (diameter 0) (color 0 0 0 0)
+  )
+  (junction (at 101.6 129.54) (diameter 0) (color 0 0 0 0)
+  )
   (junction (at 101.6 53.34) (diameter 0) (color 0 0 0 0)
-  )
-  (junction (at 88.9 93.98) (diameter 0) (color 0 0 0 0)
-  )
-  (junction (at 96.774 53.34) (diameter 0) (color 0 0 0 0)
-  )
-  (junction (at 104.14 114.3) (diameter 0) (color 0 0 0 0)
-  )
-  (junction (at 101.6 68.58) (diameter 0) (color 0 0 0 0)
-  )
-  (junction (at 101.6 144.78) (diameter 0) (color 0 0 0 0)
-  )
-  (junction (at 101.6 99.06) (diameter 0) (color 0 0 0 0)
-  )
-  (junction (at 101.6 114.3) (diameter 0) (color 0 0 0 0)
-  )
-  (junction (at 101.6 160.02) (diameter 0) (color 0 0 0 0)
-  )
-  (junction (at 104.14 83.82) (diameter 0) (color 0 0 0 0)
-  )
-  (junction (at 104.14 160.02) (diameter 0) (color 0 0 0 0)
-  )
-  (junction (at 104.14 144.78) (diameter 0) (color 0 0 0 0)
-  )
-  (junction (at 88.9 109.22) (diameter 0) (color 0 0 0 0)
-  )
-  (junction (at 101.6 129.54) (diameter 0) (color 0 0 0 0)
   )
   (junction (at 88.9 154.94) (diameter 0) (color 0 0 0 0)
@@
     (stroke (width 0) (type default) (color 255 255 0 1))
   )
-  (wire (pts (xy 96.52 53.34) (xy 96.774 53.34))
-    (stroke (width 0) (type default))
-  )
   (bus (pts (xy 121.92 38.1) (xy 121.92 40.64))
     (stroke (width 0) (type default) (color 255 255 0 1))
@@
     (stroke (width 0) (type default))
   )
+  (bus (pts (xy 121.92 132.08) (xy 121.92 147.32))
+    (stroke (width 0) (type default) (color 255 255 0 1))
+  )
+  (wire (pts (xy 104.14 160.02) (xy 104.14 165.1))
+    (stroke (width 0) (type default))
+  )
+  (wire (pts (xy 20.32 58.42) (xy 43.18 58.42))
+    (stroke (width 0) (type default))
+  )
+  (wire (pts (xy 104.14 160.02) (xy 101.6 160.02))
+    (stroke (width 0) (type default))
+  )
+  (wire (pts (xy 88.9 78.74) (xy 88.9 83.82))
+    (stroke (width 0) (type default))
+  )
+  (bus (pts (xy 121.92 101.6) (xy 121.92 116.84))
+    (stroke (width 0) (type default) (color 255 255 0 1))
+  )
+  (wire (pts (xy 86.36 63.5) (xy 88.9 63.5))
+    (stroke (width 0) (type default))
+  )
+  (wire (pts (xy 119.38 43.18) (xy 101.6 43.18))
+    (stroke (width 0) (type default) (color 255 255 0 1))
+  )
+  (wire (pts (xy 96.52 114.3) (xy 101.6 114.3))
+    (stroke (width 0) (type default))
+  )
+  (wire (pts (xy 101.6 129.54) (xy 104.14 129.54))
+    (stroke (width 0) (type default))
+  )
+  (wire (pts (xy 88.9 78.74) (xy 95.25 78.74))
+    (stroke (width 0) (type default))
+  )
+  (bus (pts (xy 83.82 121.92) (xy 83.82 137.16))
+    (stroke (width 0) (type default) (color 194 194 0 1))
+  )
+  (wire (pts (xy 104.14 53.34) (xy 104.14 68.58))
+    (stroke (width 0) (type default))
+  )
+  (wire (pts (xy 96.52 83.82) (xy 101.6 83.82))
+    (stroke (width 0) (type default))
+  )
+  (wire (pts (xy 88.9 154.94) (xy 95.25 154.94))
+    (stroke (width 0) (type default))
+  )
+  (wire (pts (xy 101.6 83.82) (xy 104.14 83.82))
+    (stroke (width 0) (type default))
+  )
+  (bus (pts (xy 71.12 73.66) (xy 71.12 76.2))
+    (stroke (width 0) (type default) (color 194 194 0 1))
+  )
+  (wire (pts (xy 101.6 99.06) (xy 104.14 99.06))
+    (stroke (width 0) (type default))
+  )
+  (wire (pts (xy 104.14 68.58) (xy 104.14 83.82))
+    (stroke (width 0) (type default))
+  )
+  (bus (pts (xy 83.82 91.44) (xy 83.82 106.68))
+    (stroke (width 0) (type default) (color 194 194 0 1))
+  )
+  (wire (pts (xy 63.5 76.2) (xy 68.58 76.2))
+    (stroke (width 0) (type default))
+  )
+  (wire (pts (xy 86.36 78.74) (xy 88.9 78.74))
+    (stroke (width 0) (type default))
+  )
+  (bus (pts (xy 121.92 99.06) (xy 121.92 101.6))
+    (stroke (width 0) (type default) (color 255 255 0 1))
+  )
+  (wire (pts (xy 35.56 43.18) (xy 35.56 48.26))
+    (stroke (width 0) (type default))
+  )
+  (wire (pts (xy 88.9 139.7) (xy 95.25 139.7))
+    (stroke (width 0) (type default))
+  )
   (wire (pts (xy 96.774 53.34) (xy 101.6 53.34))
     (stroke (width 0) (type default))
   )
-  (bus (pts (xy 121.92 132.08) (xy 121.92 147.32))
-    (stroke (width 0) (type default) (color 255 255 0 1))
-  )
-  (wire (pts (xy 104.14 160.02) (xy 104.14 165.1))
-    (stroke (width 0) (type default))
-  )
-  (wire (pts (xy 20.32 58.42) (xy 43.18 58.42))
-    (stroke (width 0) (type default))
-  )
-  (wire (pts (xy 104.14 160.02) (xy 101.6 160.02))
-    (stroke (width 0) (type default))
-  )
-  (wire (pts (xy 88.9 78.74) (xy 88.9 83.82))
-    (stroke (width 0) (type default))
-  )
-  (bus (pts (xy 121.92 101.6) (xy 121.92 116.84))
-    (stroke (width 0) (type default) (color 255 255 0 1))
-  )
-  (wire (pts (xy 86.36 63.5) (xy 88.9 63.5))
-    (stroke (width 0) (type default))
-  )
-  (wire (pts (xy 119.38 43.18) (xy 101.6 43.18))
-    (stroke (width 0) (type default) (color 255 255 0 1))
-  )
-  (wire (pts (xy 96.52 114.3) (xy 101.6 114.3))
-    (stroke (width 0) (type default))
-  )
-  (wire (pts (xy 101.6 129.54) (xy 104.14 129.54))
-    (stroke (width 0) (type default))
-  )
-  (wire (pts (xy 88.9 78.74) (xy 95.25 78.74))
-    (stroke (width 0) (type default))
-  )
-  (bus (pts (xy 83.82 121.92) (xy 83.82 137.16))
-    (stroke (width 0) (type default) (color 194 194 0 1))
-  )
-  (wire (pts (xy 104.14 53.34) (xy 104.14 68.58))
-    (stroke (width 0) (type default))
-  )
-  (wire (pts (xy 96.52 83.82) (xy 101.6 83.82))
-    (stroke (width 0) (type default))
-  )
-  (wire (pts (xy 88.9 154.94) (xy 95.25 154.94))
-    (stroke (width 0) (type default))
-  )
-  (wire (pts (xy 101.6 83.82) (xy 104.14 83.82))
-    (stroke (width 0) (type default))
-  )
-  (bus (pts (xy 71.12 73.66) (xy 71.12 76.2))
-    (stroke (width 0) (type default) (color 194 194 0 1))
-  )
-  (wire (pts (xy 101.6 99.06) (xy 104.14 99.06))
-    (stroke (width 0) (type default))
-  )
-  (wire (pts (xy 104.14 68.58) (xy 104.14 83.82))
-    (stroke (width 0) (type default))
-  )
-  (bus (pts (xy 83.82 91.44) (xy 83.82 106.68))
-    (stroke (width 0) (type default) (color 194 194 0 1))
-  )
-  (wire (pts (xy 63.5 76.2) (xy 68.58 76.2))
-    (stroke (width 0) (type default))
-  )
-  (wire (pts (xy 86.36 78.74) (xy 88.9 78.74))
-    (stroke (width 0) (type default))
-  )
-  (bus (pts (xy 121.92 99.06) (xy 121.92 101.6))
-    (stroke (width 0) (type default) (color 255 255 0 1))
-  )
-  (wire (pts (xy 35.56 43.18) (xy 35.56 48.26))
-    (stroke (width 0) (type default))
-  )
-  (wire (pts (xy 88.9 139.7) (xy 95.25 139.7))
-    (stroke (width 0) (type default))
-  )
