File: hardware/we_ssr_control/manual_control.kicad_sch (KiCad schematic)
At the start: 1 part

Commit message: Power supply changes plus misc.
Parts:
- S1: Height 9.37 -> (none); Manufacturer_Name CTS -> (none); Manufacturer_Part_Number 193-8MS -> (none)
Changed lines of the file:
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@@
   (paper "USLetter")
   (title_block
-    (date "2023-02-03")
-    (rev "0.0.10")
+    (date "2023-02-08")
+    (rev "0.0.11")
     (comment 2 "creativecommons.org/licenses/by/4.0/")
     (comment 3 "License: CC By 4.0")
@@
       (effects (font (size 1.27 1.27)) (justify left) hide)
     )
-    (property "Manufacturer_Name" "CTS" (id 12) (at 63.5 80.01 0)
-      (effects (font (size 1.27 1.27)) (justify left) hide)
-    )
-    (property "Manufacturer_Part_Number" "193-8MS" (id 13) (at 66.04 80.01 0)
-      (effects (font (size 1.27 1.27)) (justify left) hide)
-    )
-    (property "Height" "9.37" (id 14) (at 55.88 80.01 0)
-      (effects (font (size 1.27 1.27)) (justify left) hide)
-    )
+    (property "Height" "" (id 14) (at 55.88 80.01 0)
+      (effects (font (size 1.27 1.27)) (justify left) hide)
+    )

Commit message: Pre KiCad 7.0.0 WIP
Connections:
- net BANK_A.CNTL1 renamed BANK_A.OUT1
- net BANK_A.CNTL2 renamed BANK_A.OUT2
- net BANK_A.CNTL3 renamed BANK_A.OUT3
- net BANK_A.CNTL4 renamed BANK_A.OUT4
- net BANK_B.CNTL5 renamed BANK_B.OUT5
- net BANK_B.CNTL6 renamed BANK_B.OUT6
- net BANK_B.CNTL7 renamed BANK_B.OUT7
- net BANK_B.CNTL8 renamed BANK_B.OUT8
Changed lines of the file:
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@@
     (effects (font (size 1.27 1.27) bold) (justify left bottom))
   )
-  (label "BANK_A.CNTL3" (at 48.26 48.26 0)
+  (label "BANK_A.OUT3" (at 48.26 48.26 0)
     (effects (font (size 1.27 1.27)) (justify left bottom))
   )
-  (label "BANK_B.CNTL8" (at 48.26 60.96 0)
+  (label "BANK_B.OUT8" (at 48.26 60.96 0)
     (effects (font (size 1.27 1.27)) (justify left bottom))
   )
-  (label "BANK_B.CNTL5" (at 48.26 53.34 0)
+  (label "BANK_B.OUT5" (at 48.26 53.34 0)
     (effects (font (size 1.27 1.27)) (justify left bottom))
   )
-  (label "BANK_A.CNTL1" (at 48.26 43.18 0)
+  (label "BANK_A.OUT1" (at 48.26 43.18 0)
     (effects (font (size 1.27 1.27)) (justify left bottom))
   )
-  (label "BANK_B.CNTL6" (at 48.26 55.88 0)
+  (label "BANK_B.OUT6" (at 48.26 55.88 0)
     (effects (font (size 1.27 1.27)) (justify left bottom))
   )
-  (label "BANK_A.CNTL4" (at 48.26 50.8 0)
+  (label "BANK_A.OUT4" (at 48.26 50.8 0)
     (effects (font (size 1.27 1.27)) (justify left bottom))
   )
-  (label "BANK_B.CNTL7" (at 48.26 58.42 0)
+  (label "BANK_B.OUT7" (at 48.26 58.42 0)
     (effects (font (size 1.27 1.27)) (justify left bottom))
   )
-  (label "BANK_A.CNTL2" (at 48.26 45.72 0)
+  (label "BANK_A.OUT2" (at 48.26 45.72 0)
     (effects (font (size 1.27 1.27)) (justify left bottom))
   )
-  (hierarchical_label "BANK_A{CNTL[1..4]}" (shape passive) (at 76.2 38.1 0)
+  (hierarchical_label "BANK_A{OUT1..4]}" (shape passive) (at 76.2 38.1 0)
     (effects (font (size 2 2) bold) (justify left))
   )
-  (hierarchical_label "BANK_B{CNTL[5..8]}" (shape passive) (at 76.2 66.04 0)
+  (hierarchical_label "BANK_B{OUT[5..8]}" (shape passive) (at 76.2 66.04 0)
     (effects (font (size 2 2) bold) (justify left))
   )
