File: hardware/we_ssr_control/manual_control.kicad_sch (KiCad schematic)
At the start: 1 part

Commit message: Commit before removing git submodules
Changed lines of the file:
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@@
     (effects (font (size 1.27 1.27)) (justify left bottom))
   )
-  (hierarchical_label "BANK_A{OUT1..4]}" (shape passive) (at 76.2 38.1 0) (fields_autoplaced)
+  (hierarchical_label "BANK_A{OUT[1..4]}" (shape passive) (at 76.2 38.1 0) (fields_autoplaced)
     (effects (font (size 2 2) bold) (justify left))
   )
